File: epdiy-v7/epaper-breakout.kicad_pcb (KiCad board)
At the start: 4 copper layers, 100 x 55 mm, 118 parts, among them J1 USB_C_Receptacle_USB2.0, J2 EXTENSION_HEADER, J3 USB_HDR, J4 XF2M-3315-1A, J5 CONN_BAT, J6 8BIT_HEADER, J7 ESP_HDR, Q1 AO3401A, Q3 MMBT3904, Q4 MMBT3904, U1 RT9080-33GJ5, U10 ED060XC5, U11 TP4056, U2 PCA9535PW, U3 TPS651851RSLR, U4 USBLC6-2P6, U5 XC6206PxxxMR, U6 ED078KH6, U7 PCF8563T, U8 ESP32-S3-WROOM-1, U9 CH340C, Y1 32.768K

Commit message: epdiy v7 cleanup
Parts:
- U9: renamed from U3; value TPS651851RSLR -> RSL48_4P4X4P4
- renumbered REF** to #SYM101, C38 to C1, C24 to C11, C7 to C12, C5 to C13, C12 to C14, C2 to C15, C9 to C16, C13 to C17, C20 to C18, C6 to C19, C35 to C2, C27 to C20, C30 to C21, C4 to C22, C1 to C23, C3 to C24, C29 to C25, C8 to C26, C33 to C27, C25 to C28, C11 to C29, C41 to C3, C26 to C30, C28 to C31, C31 to C32, C15 to C33, C17 to C34, C19 to C35, C16 to C37, C22 to C38, C32 to C39, C21 to C4, C18 to C40, C23 to C41, C34 to C42, C37 to C5, C39 to C6, C40 to C7, C42 to C8, C14 to C9, D9 to D10, D10 to D2, D7 to D3, D3 to D4, D2 to D5, D5 to D7, D4 to D8, D8 to D9, H4 to H1, H1 to H2, H2 to H3, H3 to H4, J2 to J1, J7 to J2, J4 to J3, J3 to J4, J1 to J5, J5 to J6, J6 to J7, JP2 to JP1, JP1 to JP2, Q3 to Q1, Q4 to Q2, Q1 to Q3, R30 to R1, R11 to R10, R14 to R11, R6 to R12, R32 to R13, R4 to R14, R2 to R15, R31 to R16, R9 to R17, R20 to R18, R27 to R2, R24 to R20, R23 to R21, R18 to R22, R10 to R23, R21 to R24, R3 to R25, R8 to R26, R28 to R27, R22 to R28, R26 to R29, R5 to R3, R33 to R4, R29 to R5, R7 to R6, R16 to R7, R15 to R8, R1 to R9, TP3 to TP1, TP1 to TP2, TP2 to TP3, U10 to U1, U8 to U10, U9 to U3, U7 to U5, U5 to U6, U6 to U7, U1 to U8
Other:
- board text removed: "EPD3.3V"
