File: epdiy-v7/epaper-breakout.kicad_sch (KiCad schematic)
At the start: 117 parts, among them J1 USB_C_Receptacle_USB2.0, J2 EXTENSION_HEADER, J3 USB_HDR, J4 XF2M-3315-1A, J5 CONN_BAT, J6 8BIT_HEADER, J7 ESP_HDR, Q1 AO3401A, Q3 MMBT3904, Q4 MMBT3904, U1 RT9080-33GJ5, U10 ED060XC5, U11 TP4056, U2 PCA9535PW, U3 TPS651851RSLR, U4 USBLC6-2P6, U5 XC6206PxxxMR, U6 ED078KH6, U7 PCF8563T, U8 ESP32-S3-WROOM-1, U9 CH340C, Y1 32.768K

Commit message: epdiy v7 cleanup
Parts:
- C17: LCSC C16133 -> C16133
- D10: LCSC C8598 -> C8598
- D9: LCSC C84256 -> C84256
- J2: symbol Connector:Conn_01x13_Female -> Connector:Conn_01x13_Socket
- J3, J5: symbol Connector:Conn_01x02_Female -> Connector:Conn_01x02_Socket
- J6: symbol Connector:Conn_01x10_Female -> Connector:Conn_01x10_Socket
- J7: symbol Connector:Conn_01x12_Female -> Connector:Conn_01x12_Socket
- L1: LCSC C222947 -> C222947
- U11: LCSC C16581 -> C16581
Other:
- moved on the sheet: C2, C3, C41, J5, R4, R6, U1
