File: epdiy-v7/epdiy-v7.kicad_sch (KiCad schematic)
At the start: 117 parts, among them J1 USB_C_Receptacle_USB2.0, J2 EXTENSION_HEADER, J3 USB_HDR, J4 XF2M-3315-1A, J5 CONN_BAT, J6 8BIT_HEADER, J7 ESP_HDR, Q1 AO3401A, Q3 MMBT3904, Q4 MMBT3904, U1 RT9080-33GJ5, U10 ED060XC5, U11 TP4056, U2 PCA9535PW, U3 TPS651851RSLR, U4 USBLC6-2P6, U5 XC6206PxxxMR, U6 ED078KH6, U7 PCF8563T, U8 ESP32-S3-WROOM-1, U9 CH340C, Y1 32.768K

Commit message: epdiy v7: exclude non-parts from BoM
Parts:
- H1, H2, H3, H4, J2, J3, J5, J6, J7, JP1, JP2, TP1, TP2, TP3, TP4, TP5: now left out of the parts list
