File: extension-cable/extension-cable.kicad_pcb (KiCad board)
At the start: 2 copper layers, 32 x 37.1 mm, 4 parts, among them J1 XF2M-3315-1A, J2 XF2M-3315-1A

Commit message: migrate extension cable to kicad 7
Other:
- net class Default removed
