File: epaper-breakout/epaper-breakout.kicad_pcb (KiCad board)
At the start: 4 copper layers, 100 x 45 mm, 109 parts, among them J1 XF2M-3315-1A, J2 C10418, J3 Conn_02x05_Counter_Clockwise, J4 ED060SC4, J5 Conn_01x02_Female, J7 Conn_01x12, Q3 MMBT3904, Q4 MMBT3904, U1 MCP1700-3302E_SOT23, U11 TP4056, U12 CH340C, U2 PCA9535PW, U3 TPS651851RSLR, U4 XC6206PxxxMR, U5 ESP32-WROVER, U6 ED060XC5, U7 TPS2113APW

Commit message: update v6 pcb to kicad 7
Parts:
- C15, C16, C21, C22, C23, C39, C40: value 0.1uF -> 100nF
- TH1: value 10k -> 10k/3380K
- moved Q4 0.45 mm to (39.7, 36.8)
Connections:
- net /~DTR renamed /~{DTR}
- net /~GPIO_INTR renamed /~{GPIO_INTR}
- net /~RTS renamed /~{RTS}
- J1 pad 2: Net-(J1-Pad2) -> unconnected-(J1-NC-Pad2)
- J1 pad 21: Net-(J1-Pad21) -> unconnected-(J1-NC-Pad21)
- J1 pad 23: Net-(J1-Pad23) -> unconnected-(J1-NC-Pad23)
- J1 pad 25: Net-(J1-Pad25) -> unconnected-(J1-NC-Pad25)
- J1 pad 27: Net-(J1-Pad27) -> unconnected-(J1-NC-Pad27)
- J1 pad 34: Net-(J1-Pad34) -> unconnected-(J1-CASE_1-Pad34)
- J1 pad 35: Net-(J1-Pad35) -> unconnected-(J1-CASE_2-Pad35)
- J1 pad 4: Net-(J1-Pad4) -> unconnected-(J1-NC-Pad4)
- J1 pad 6: Net-(J1-Pad6) -> unconnected-(J1-NC-Pad6)
- J2 pad 4: Net-(J2-Pad4) -> unconnected-(J2-ID-Pad4)
- J4 pad 20: Net-(J4-Pad20) -> unconnected-(J4-NC-Pad20)
- J4 pad 21: Net-(J4-Pad21) -> unconnected-(J4-NC-Pad21)
- J4 pad 25: Net-(J4-Pad25) -> unconnected-(J4-NC-Pad25)
- J4 pad 26: Net-(J4-Pad26) -> unconnected-(J4-NC-Pad26)
- J4 pad 39: Net-(J4-Pad39) -> unconnected-(J4-NC-Pad39)
- U11 pad 9: Net-(U11-Pad9) -> unconnected-(U11-PP-Pad9)
- U12 pad 10: Net-(U12-Pad10) -> unconnected-(U12-~{DSR}-Pad10)
- U12 pad 11: Net-(U12-Pad11) -> unconnected-(U12-~{RI}-Pad11)
- U12 pad 12: Net-(U12-Pad12) -> unconnected-(U12-~{DCD}-Pad12)
- U12 pad 15: Net-(U12-Pad15) -> unconnected-(U12-R232-Pad15)
- U12 pad 7: Net-(U12-Pad7) -> unconnected-(U12-NC-Pad7)
- U12 pad 8: Net-(U12-Pad8) -> unconnected-(U12-NC-Pad8)
- U12 pad 9: Net-(U12-Pad9) -> unconnected-(U12-~{CTS}-Pad9)
- U3 pad 11: Net-(U3-Pad11) -> unconnected-(U3-NC-Pad11)
- U3 pad 13: Net-(U3-Pad13) -> unconnected-(U3-NC-Pad13)
- U3 pad 20: Net-(U3-Pad20) -> unconnected-(U3-NC-Pad20)
- U3 pad 38: Net-(U3-Pad38) -> unconnected-(U3-NC-Pad38)
- U3 pad 39: Net-(U3-Pad39) -> unconnected-(U3-NC-Pad39)
- U5 pad 17: Net-(U5-Pad17) -> unconnected-(U5-SD2_IO9-Pad17)
- U5 pad 18: Net-(U5-Pad18) -> unconnected-(U5-SD3_IO10-Pad18)
- U5 pad 19: Net-(U5-Pad19) -> unconnected-(U5-CMD_IO11-Pad19)
- U5 pad 20: Net-(U5-Pad20) -> unconnected-(U5-CLK_IO6-Pad20)
- U5 pad 21: Net-(U5-Pad21) -> unconnected-(U5-SD0_IO7-Pad21)
- U5 pad 22: Net-(U5-Pad22) -> unconnected-(U5-SD1_IO8-Pad22)
- U5 pad 27: Net-(U5-Pad27) -> unconnected-(U5-IO16-Pad27)
- U5 pad 28: Net-(U5-Pad28) -> unconnected-(U5-IO17-Pad28)
- U5 pad 32: Net-(U5-Pad32) -> unconnected-(U5-NC-Pad32)
- U6 pad 22: Net-(U6-Pad22) -> unconnected-(U6-NC-Pad22)
- U6 pad 23: Net-(U6-Pad23) -> unconnected-(U6-NC-Pad23)
- U6 pad 24: Net-(U6-Pad24) -> unconnected-(U6-NC-Pad24)
- U6 pad 25: Net-(U6-Pad25) -> unconnected-(U6-NC-Pad25)
- U6 pad 30: Net-(U6-Pad30) -> unconnected-(U6-NC-Pad30)
- U6 pad 4: Net-(U6-Pad4) -> unconnected-(U6-NC-Pad4)
- U6 pad 5: Net-(U6-Pad5) -> unconnected-(U6-NC-Pad5)
- U7 pad 1: Net-(U7-Pad1) -> unconnected-(U7-STAT-Pad1)
Routing:
- net GND: track 295.2 -> 292.0 mm, vias 135 -> 134
- net /~{DTR}: track 12.4 -> 14.7 mm
Other:
- net class Default removed
