File: adapters/9.7_40_to_34_6inch/9.7_40_to_34_6inch.kicad_pcb (KiCad board)
At the start: 2 copper layers, 64.8 x 37 mm, 8 parts, among them J1 XF2M-3315-1A, U1 ED060XC5, U2 ED078KH6, U3 ED060XC5

Commit message: Fixes #5
Parts:
- removed H3, H4: MountingHole, MountingHole:MountingHole_2.2mm_M2
- removed J1: XF2M-3315-1A, footprints:FH1233S05SH55
- removed U3: ED060XC5, epaper-breakout:X05A20H34G
Routing:
- net /CKV_A: track 52.9 -> 0.00 mm, vias 2 -> 0
- net EPD_VDD_A: track 51.6 -> 0.00 mm
- net /EP_MODE_A: track 43.7 -> 0.00 mm, vias 2 -> 0
- net /-15V_A: track 42.5 -> 0.00 mm, vias 2 -> 0
- net /+22V_A: track 38.2 -> 0.00 mm, vias 2 -> 0
- net /BORDER_A: track 34.2 -> 0.00 mm, vias 2 -> 0
- net /EP_STV_A: track 33.6 -> 0.00 mm, vias 2 -> 0
- net /XCL_A: track 25.3 -> 0.00 mm
- net /LEH_A: track 24.9 -> 0.00 mm, vias 2 -> 0
- net /EP_VCOM_A: track 24.9 -> 0.00 mm, vias 2 -> 0
- net /EP_OE_A: track 24.3 -> 0.00 mm, vias 2 -> 0
- net /XSTL_A: track 23.9 -> 0.00 mm, vias 2 -> 0
- net /D0_A: track 23.7 -> 0.00 mm, vias 2 -> 0
- net /D7_A: track 23.2 -> 0.00 mm, vias 2 -> 0
- net /D1_A: track 23.1 -> 0.00 mm, vias 2 -> 0
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Other:
- board size 64.8 x 37 mm -> 32 x 37 mm
- board text removed: "33"
- board text removed: "33 pin 9.7{dblquote}"
- board text removed: "9.7{dblquote} to 6{dblquote} ADAPTER"
