File: adapters/9.7_40_to_34_6inch/9.7_40_to_34_6inch.kicad_sch (KiCad schematic)
At the start: 8 parts, among them J1 XF2M-3315-1A, U1 ED060XC5, U2 ED078KH6, U3 ED060XC5

Commit message: Fixes #5
Parts:
- removed J1: XF2M-3315-1A, footprints:FH1233S05SH55, symbol epd_breakout:XF2M-3315-1A
- removed U3: ED060XC5, epaper-breakout:X05A20H34G, symbol epd_breakout:ED060XC5
Connections:
- no-connect marks 10 -> 8
Other:
- note added: "ADAPTER 40->34"
- note removed: "1st connector A 33->34"
- note removed: "2nd connector B 40->34"
- note removed: "EPD Connector 33pin, 8bit"
- moved on the sheet: H1, H2, H3, H4, U1, U2
