File: epdiy-v7-raw/epdiy-v7-raw.kicad_pcb (KiCad board)
At the start: 4 copper layers, 128.4 x 74.9 mm, 118 parts, among them CN1 WP27D-S050VA3-R15000, IC1 MPU-6500, J1 USB_C_Receptacle_USB2.0, J2 EXTENSION_HEADER, J3 SIGNALS_HEADER, J5 CONN_BAT, J6 THD2528-11SD-GF, J7 ESP_HDR, Q1 AO3401A, SW1 TC-0522C-1.7-160G, SW2 TC-0522C-1.7-160G, SW3 K2-1806SQ-A2DW-04, SW4 K2-1806SQ-A2DW-04, SW5 K2-1806SQ-A2DW-04, U1 RT9080-33GJ5, U10 ED060XC5, U11 TP4056, U3 TPS651851RSLR, U4 USBLC6-2P6, U8 ESP32-S3-WROOM-1, Y1 RV-3032-C7

Commit message: 1.1 is ready
Parts:
- removed C16: 10uF, Capacitor_SMD:C_0805_2012Metric
- removed C21: 22pF, Capacitor_SMD:C_0402_1005Metric
- removed J7: ESP_HDR, Connector_PinHeader_2.54mm:PinHeader_1x11_P2.54mm_Vertical
- removed JP1: VBAT_GPIO1, Jumper:SolderJumper-2_P1.3mm_Bridged2Bar_Pad1.0x1.5mm
- removed SW2: TC-0522C-1.7-160G, footprints:C2845289_SW-SMD_4P-L5.2-W5.2-P3.70-LS6.4
- C15: value 100nF -> 22pF
- J5: value CONN_BAT -> S2B-PH-SM4-TB_LF__SN_; footprint Connector_PinHeader_2.54mm:PinHeader_1x02_P2.54mm_Vertical -> footprints:S2BPHSM4TBLFSN
- JP2: footprint Jumper:SolderJumper-2_P1.3mm_Bridged2Bar_Pad1.0x1.5mm -> Jumper:SolderJumper-2_P1.3mm_Open_Pad1.0x1.5mm
- R12: value 10K -> 1k
- R3: value 2.4k -> 5.1k
- moved J5 5.97 mm to (79.0, 90.6), turned to 0 degrees
- moved JP2 3.66 mm to (92.1, 75.8), turned to -135 degrees
- moved R5 3.27 mm to (117.7, 93.0), turned to 180 degrees
- moved R21 0.61 mm to (66.3, 115.5)
- moved C23 0.28 mm to (68.9, 118.4)
- moved C3 0.09 mm to (113.1, 104.8), turned to 0 degrees
Connections:
- C15 pad 1: /EN -> GND
- C15 pad 2: GND -> /IO0
- C23 pad 2: Net-(JP1-B) -> /GPIO_1
- J2 pad 3: /SDA -> /SCL
- J2 pad 4: /SCL -> /SDA
- J6 pad 2: /GPIO_36 -> /SD_CS
- J6 pad 3: /GPIO_35 -> /SD_CMD
- J6 pad 7: /IO0 -> /GPIO_2
- J6 pad 9: /GPIO_37 -> unconnected-(J6-CD-Pad9)
- R21 pad 2: Net-(JP1-B) -> /GPIO_1
- R22 pad 1: Net-(JP1-B) -> /GPIO_1
- RN1 pad 1: /IO0 -> /GPIO_2
- RN1 pad 3: /GPIO_35 -> /SD_CMD
- RN1 pad 4: /GPIO_36 -> /SD_CS
- SW3 pad 2: /GPIO_3 -> /IO0
- U8 pad 36: TX -> /SD_CS
- U8 pad 37: RX -> /SD_CMD
Routing:
- net /GPIO_3: track 173.2 -> 54.3 mm, vias 4 -> 2
- net /GPIO_37: track 116.4 -> 0.00 mm, vias 2 -> 0
- net /GPIO_36: track 113.3 -> 0.00 mm, vias 2 -> 0
- net /GPIO_35: track 96.0 -> 0.00 mm, vias 2 -> 0
- net /SD_CMD: track 0.00 -> 78.5 mm, vias 0 -> 2
- net /SD_CS: track 0.00 -> 72.9 mm, vias 0 -> 2
- net Net-(JP1-B): track 54.8 -> 0.00 mm, vias 2 -> 0
- net /GPIO_2: track 86.6 -> 122.6 mm
- net /GPIO_46: track 127.9 -> 100.8 mm
- net /GPIO_1: track 91.9 -> 67.5 mm
- net GND: track 213.9 -> 202.2 mm, vias 102 -> 100
- net /IO0: track 94.8 -> 84.3 mm
- net /RTC_INT: track 36.9 -> 31.6 mm
- net 3.3V: track 146.0 -> 150.9 mm, vias 15 -> 14
- net /SCL: track 155.1 -> 150.8 mm
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Other:
- board text added: "1 ADC"
- board text added: "OSPI"
- board text removed: "BOOT"
- board text removed: "CLK"
- board text removed: "IO35"
- board text removed: "IO36"
- board text removed: "IO37"
- board text removed: "RTCI-IO2"
- board text removed: "VBAT-IO1"
