File: epdiy-v7-model-F/epaper-breakout.kicad_pcb (KiCad board)
At the start: 4 copper layers, 100 x 55 mm, 124 parts, among them J1 USB_C_Receptacle_USB2.0, J2 EXTENSION_HEADER, J3 SM04B-SRSS-TB_LF__SN_, J4 XF2M-3315-1A, J5 CONN_BAT, J6 8BIT_HEADER, J7 ESP_HDR, J8 ED133UT2, J9 USB_C_Receptacle_USB2.0, Q1 AO3401A, Q3 MMBT3904, Q4 MMBT3904, U1 MCP1700-3302E_SOT23, U10 MCP1700-3302E_SOT23, U11 TP4056, U2 PCA9535PW, U3 TPS651851RSLR, U4 USBLC6-2P6, U5 XC6206PxxxMR, U6 ED078KH6, U7 LP5240HVF, U8 ESP32-S3-WROOM-1, U9 CH340C, Y1 RV-3032-C7

Commit message: 1.0 under review
Parts:
- removed TP7: RTC_VBACKUP, TestPoint:TestPoint_Pad_D1.5mm
- added C43: superCAP, footprints:C9900013866_SUPERCAP-TH_XH414HG, F.Cu at (80.9, 36.4)
- added JP3: 3V3_JOIN, Jumper:SolderJumper-2_P1.3mm_Open_RoundedPad1.0x1.5mm, F.Cu at (83.7, 29.3)
- moved C21 2.40 mm to (86.9, 34.0), turned to 0 degrees
Routing:
- net Net-(Y1-VBACKUP): track 8.87 -> 2.40 mm, vias 2 -> 0
- net QWIIC_3V3: track 4.70 -> 8.95 mm
- net /SCL: track 119.7 -> 123.6 mm
- net GND: track 211.7 -> 215.6 mm
- net 3.3V: track 107.0 -> 108.6 mm, vias 16 -> 17
Other:
- board text added: "C9900013866"
- board text added: "HIGH ▲ for 3V3 extra power"
- board text added: "Joins U10 250mA ▴ w/general 3V3"
- board text removed: "BAT BACKUP"

Commit message: Final touches F model
Parts:
- removed U7: LP5240HVF, footprints:C2890373_WLCSP-4
- U10: value MCP1700-3302E_SOT23 -> RT9080-33GJ5; footprint Package_TO_SOT_SMD:SOT-23 -> Package_TO_SOT_SMD:TSOT-23-5
- U6: footprint Connector_FFC-FPC:Hirose_FH12-40S-0.5SH_1x40-1MP_P0.50mm_Horizontal -> footprints:FH1240S05SH55
- moved C21 2.24 mm to (89.0, 34.6), turned to -135 degrees
- moved U10 1.29 mm to (90.6, 30.6), turned to 90 degrees
Connections:
- C21 pad 1: /QWIIC_VIN -> VIN
- U10 pad 1: GND -> VIN
- U10 pad 2: QWIIC_3V3 -> unconnected-(U10-GND-Pad2)
- U10 pad 3: /QWIIC_VIN -> /GPIO_46
Routing:
- net /GPIO_46: track 53.4 -> 65.3 mm
- net /QWIIC_VIN: track 7.44 -> 0.00 mm, vias 2 -> 0
- net GND: track 215.6 -> 212.2 mm, vias 114 -> 113
- net VIN: track 120.4 -> 118.6 mm
- net QWIIC_3V3: track 8.95 -> 9.92 mm
Other:
- board text added: "Joins U10 500mA ▴ w/general 3V3"
- board text added: "epdiy v7_10.3{dblquote}"
- board text removed: "Joins U10 250mA ▴ w/general 3V3"
- board text removed: "epdiy v7"
