File: epdiy-v7-model-F/epaper-breakout.kicad_sch (KiCad schematic)
At the start: 123 parts, among them J1 USB_C_Receptacle_USB2.0, J2 ED133UT2, J2 EXTENSION_HEADER, J3 SM04B-SRSS-TB_LF__SN_, J4 XF2M-3315-1A, J5 CONN_BAT, J6 8BIT_HEADER, J7 ESP_HDR, J9 USB_C_Receptacle_USB2.0, Q1 AO3401A, Q3 MMBT3904, Q4 MMBT3904, U1 MCP1700-3302E_SOT23, U10 MCP1700-3302E_SOT23, U11 TP4056, U2 PCA9535PW, U3 TPS651851RSLR, U4 USBLC6-2P6, U5 XC6206PxxxMR, U6 ED078KH6, U7 LP5240HVF, U8 ESP32-S3-WROOM-1, U9 CH340C, Y1 RV-3032-C7

Commit message: 1.0 under review
Parts:
- removed TP7: RTC_VBACKUP, TestPoint:TestPoint_Pad_D1.5mm, symbol Connector:TestPoint
- added C43: superCAP, footprints:C9900013866_SUPERCAP-TH_XH414HG, symbol Device:C_Polarized
- added JP3: 3V3_JOIN, Jumper:SolderJumper-2_P1.3mm_Open_RoundedPad1.0x1.5mm, symbol Jumper:Jumper_2_Open
Connections:
- net 3.3V: now also JP3.2 (B)
- net GND: now also C43.2
- net QWIIC_3V3: now also JP3.1 (A)
- net at Y1.1 (VBACKUP): now also C43.1

Commit message: Final touches F model
Parts:
- removed U10: MCP1700-3302E_SOT23, Package_TO_SOT_SMD:SOT-23, symbol epaper-breakout-rescue:MCP1700-3302E_SOT23-Regulator_Linear
- removed U7: LP5240HVF, footprints:C2890373_WLCSP-4, symbol easyeda:LP5240HVF
- added U10: RT9080-33GJ5, Package_TO_SOT_SMD:TSOT-23-5, symbol epdiy:RT9080-33GJ5
- renumbered J2 to J8
Connections:
- net QWIIC_VIN is gone; now on net VIN: C21.1
- net GPIO_46: now also U10.3 (EN)
- net QWIIC_3V3: now also U10.5 (VOUT)
- net VIN: now also U10.1 (VIN)
Other:
- moved on the sheet: C21, C39, JP3
