File: epdiy-v7-light/epdiy-v7-light.kicad_sch (KiCad schematic)
At the start: 115 parts, among them IC1 TPS2117DRLR, IC2 BQ27426YZFR, J2 EXTENSION_HEADER, J3 SM04B-SRSS-TB_LF__SN_, J4 Conn_01x02_Shielded, J6 8BIT_HEADER, J9 USB_C_Receptacle_USB2.0, Q2 CPH3350, Q3 NTR4170NT1G, Q4 CPH3350, SW1 HX-3X6X3.5-CA-0.6-2.5N, SW2 HX-3X6X3.5-CA-0.6-2.5N, SW3 HX-3X6X3.5-CA-0.6-2.5N, SW4 HX-3X6X3.5-CA-0.6-2.5N, U1 MCP1700-3302E_SOT23, U10 RT9080-33GJ5, U11 TP4056, U2 PCA9535PW, U3 TPS651851RSLR, U4 DS3231MZ, U6 ED078KH6, U8 ESP32-S3-WROOM-1

Commit message: Add v7-light
Parts:
- removed C41: 22uF, footprints:C140412_CAP-SMD_L3.5-W2.8, symbol Device:C_Polarized
Connections:
- net 3.3V is gone; now on net +3V3: C17.1, C18.2, C3.2, C40.1, J2.2 (Pin_2), JP3.2 (B), R10.2, R14.1, R15.2, R16.1, R33.1, R4.1, R6.1, U1.2 (VO), U2.24 (VDD), U3.45 (VIN3P3), U8.2 (3V3)
Other:
- moved on the sheet: C17, C18, R4, R6
