File: epdiy-v7-light/epdiy-v7-light.kicad_sch (KiCad schematic)
At the start: 114 parts, among them IC1 TPS2117DRLR, IC2 BQ27426YZFR, J2 EXTENSION_HEADER, J3 SM04B-SRSS-TB_LF__SN_, J4 Conn_01x02_Shielded, J6 8BIT_HEADER, J9 USB_C_Receptacle_USB2.0, Q2 CPH3350, Q3 NTR4170NT1G, Q4 CPH3350, SW1 HX-3X6X3.5-CA-0.6-2.5N, SW2 HX-3X6X3.5-CA-0.6-2.5N, SW3 HX-3X6X3.5-CA-0.6-2.5N, SW4 HX-3X6X3.5-CA-0.6-2.5N, U1 MCP1700-3302E_SOT23, U10 RT9080-33GJ5, U11 TP4056, U2 PCA9535PW, U3 TPS651851RSLR, U4 DS3231MZ, U6 ED078KH6, U8 ESP32-S3-WROOM-1

Commit message: v7 light 10.3
Parts:
- removed J6: 8BIT_HEADER, Connector_PinHeader_2.54mm:PinHeader_1x10_P2.54mm_Vertical, symbol Connector:Conn_01x10_Female
- added C41: 22pF, Capacitor_SMD:C_0402_1005Metric, symbol Device:C
- added SW5: HX-3X6X3.5-CA-0.6-2.5N, footprints:SW-SMD_HX-3X6X3.5-CA-0.6-2.5N, symbol easyeda:HX-3X6X3.5-CA-0.6-2.5N
- added SW6: MK-12C02-G015, footprints:C2911519_switch-MK-12C02-G020, symbol EASY:MK-12C02-G015
Connections:
- net VBUS is gone; now on net +VBUS: D10.2 (A), J9.A4 (VBUS), J9.A9 (VBUS), J9.B4 (VBUS), J9.B9 (VBUS)
- net +BATT: now also J4.1 (Pin_1), SW6.3
- net +BATT_INPUT: no longer J4.1 (Pin_1)
- net BTN_SELECT: now also U8.16 (GPIO46); no longer U8.39 (GPIO1/TOUCH1/ADC1_CH0)
- net CKV: now also U8.25 (GPIO48/SPICLK_N/SUBSPICLK_N_DIFF); no longer U8.35 (MTMS/GPIO42)
- net D0: now also U8.5 (GPIO5/TOUCH5/ADC1_CH4); no longer U8.24 (GPIO47/SPICLK_P/SUBSPICLK_P_DIFF)
- net D1: now also U8.6 (GPIO6/TOUCH6/ADC1_CH5); no longer U8.23 (GPIO21)
- net D10: now also U8.19 (GPIO11/TOUCH11/ADC2_CH0/FSPID/FSPIIO5/SUBSPID); no longer U8.10 (GPIO17/U1TXD/ADC2_CH6)
- net D11: now also U8.20 (GPIO12/TOUCH12/ADC2_CH1/FSPICLK/FSPIIO6/SUBSPICLK); no longer U8.9 (GPIO16/U0CTS/ADC2_CH5/XTAL_32K_NH5)
- net D12: now also U8.21 (GPIO13/TOUCH13/ADC2_CH2/FSPIQ/FSPIIO7/SUBSPIQ); no longer U8.8 (GPIO15/U0RTS/ADC2_CH4/XTAL_32K_P)
- net D13: now also U8.22 (GPIO14/TOUCH14/ADC2_CH3/FSPIWP/FSPIDQS/SUBSPIWP); no longer U8.7 (GPIO7/TOUCH7/ADC1_CH6)
- net D14: now also U8.23 (GPIO21); no longer U8.6 (GPIO6/TOUCH6/ADC1_CH5)
- net D15: now also U8.24 (GPIO47/SPICLK_P/SUBSPICLK_P_DIFF); no longer U8.5 (GPIO5/TOUCH5/ADC1_CH4)
- net D2: now also U8.7 (GPIO7/TOUCH7/ADC1_CH6); no longer U8.22 (GPIO14/TOUCH14/ADC2_CH3/FSPIWP/FSPIDQS/SUBSPIWP)
- net D3: now also U8.8 (GPIO15/U0RTS/ADC2_CH4/XTAL_32K_P); no longer U8.21 (GPIO13/TOUCH13/ADC2_CH2/FSPIQ/FSPIIO7/SUBSPIQ)
- net D4: now also U8.9 (GPIO16/U0CTS/ADC2_CH5/XTAL_32K_NH5); no longer U8.20 (GPIO12/TOUCH12/ADC2_CH1/FSPICLK/FSPIIO6/SUBSPICLK)
- net D5: now also U8.10 (GPIO17/U1TXD/ADC2_CH6); no longer U8.19 (GPIO11/TOUCH11/ADC2_CH0/FSPID/FSPIIO5/SUBSPID)
- net D6: now also U8.11 (GPIO18/U1RXD/ADC2_CH7/CLK_OUT3); no longer U8.18 (GPIO10/TOUCH10/ADC1_CH9/FSPICS0/FSPIIO4/SUBSPICS0)
- net D7: now also U8.12 (GPIO8/TOUCH8/ADC1_CH7/SUBSPICS1); no longer U8.17 (GPIO9/TOUCH9/ADC1_CH8/FSPIHD/SUBSPIHD)
- net D8: now also U8.17 (GPIO9/TOUCH9/ADC1_CH8/FSPIHD/SUBSPIHD); no longer U8.12 (GPIO8/TOUCH8/ADC1_CH7/SUBSPICS1)
- net D9: now also U8.18 (GPIO10/TOUCH10/ADC1_CH9/FSPICS0/FSPIIO4/SUBSPICS0); no longer U8.11 (GPIO18/U1RXD/ADC2_CH7/CLK_OUT3)
- net EP_STV: now also U8.26 (GPIO45); no longer U8.34 (MTDI/GPIO41/CLK_OUT1)
- net GND: now also C41.1, SW5.1
- net IO0: now also C41.2, SW5.2
- net LEH: now also U8.35 (MTMS/GPIO42); no longer U8.25 (GPIO48/SPICLK_N/SUBSPICLK_N_DIFF)
- net PWR_STATE: now also U2.6 (IO0_2); no longer U8.15 (GPIO3/TOUCH3/ADC1_CH2)
- net RTC_INT: now also U8.39 (GPIO1/TOUCH1/ADC1_CH0)
- net VIN2: now also SW6.2
- net XSTL: now also U8.34 (MTDI/GPIO41/CLK_OUT1); no longer U8.26 (GPIO45)
- net GPIO_46 renamed QWIIC_PWR_EN
- net QWIIC_PWR_EN: now also U8.15 (GPIO3/TOUCH3/ADC1_CH2); no longer U8.16 (GPIO46)
- no-connect marks 15 -> 26
Other:
- note added: "IO0 BOOT / USR BUTON"
- note removed: "*"
- note removed: "Breakout Header for unused pins in 8bit mode"
- moved on the sheet: C13, C15, J2, J9, Q2, Q3, Q4, R10, R11, R12, R13, R15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
